File: hardware/a33.kicad_sch (KiCad schematic)
At the start: 1 part, among them U1 A33

Commit message: Update
Parts:
- added C25, C26: 100n, Capacitor_SMD:C_0201_0603Metric, symbol Device:C_Small
- added R10, R9: 1k, Resistor_SMD:R_0201_0603Metric, symbol Device:R_Small
- added R6: 240, Resistor_SMD:R_0201_0603Metric, symbol Device:R_Small
Connections:
- net +1V5: now also C25.1, R9.1
- net GND: now also C26.2, R10.2, R6.2
- net A6: now reaches U1.A1 (DA6)
- net A8: now reaches U1.B1 (DA8)
- net A14: now reaches U1.C1 (DA14)
- net A11: now reaches U1.C2 (DA11)
- net A1: now reaches U1.D1 (DA1)
- net A4: now reaches U1.D2 (DA4)
- net A12: now reaches U1.E1 (DA12)
- net A10: now reaches U1.E2 (DA10)
- net A15: now reaches U1.E3 (DA15)
- net A0: now reaches U1.E4 (DA0)
- net A5: now reaches U1.F1 (DA5)
- net A2: now reaches U1.F2 (DA2)
- net A13: now reaches U1.F3 (DA13)
- net A9: now reaches U1.F4 (DA9)
- net CLK+: now reaches U1.G1 (DCK)
- net CLK-: now reaches U1.G2 (DCKB)
- net ~{RESET}: now reaches U1.G3 (DRST)
- net A7: now reaches U1.G4 (DA7)
- net A3: now reaches U1.H3 (DA3)
- net BA2: now reaches U1.H4 (DBA2)
- net BA0: now reaches U1.J3 (DBA0)
- net CKE0: now reaches U1.J4 (DCKE)
- net DQS0-: now reaches U1.K1 (DQS0B)
- net DQS0+: now reaches U1.K2 (DQS0)
- net ~{WE}: now reaches U1.K3 (DWE)
- net BA1: now reaches U1.K4 (DBA1)
- net ODT0: now reaches U1.L3 (DODT)
- net ~{RAS}: now reaches U1.L4 (DRAS)
- net ODT1: now reaches U1.L7 (DODT1)
- net ~{CAS}: now reaches U1.M3 (DCAS)
- net DQM0: now reaches U1.N2 (DQM0)
- net ~{CS0}: now reaches U1.N3 (DCS)
- net ~{CS1}: now reaches U1.N5 (DCS1)
- net CKE1: now reaches U1.N7 (DCKE1)
- net DQS1+: now reaches U1.R1 (DQS1)
- net at U1.R3 (DZQ): now also R6.1
- net DQS1-: now reaches U1.T1 (DQS1B)
- net DQM1: now reaches U1.T3 (DQM1)
- new net: C25.2, C26.1, R10.1, R9.2, U1.M4 (DVREF)
Other:
- note added: "243?"
- note added: "Pull up/down?"
